File: examples/royalblue54l-feather/sch/nPM1300.kicad_sch (KiCad schematic)
At the start: 13 parts, among them U2 nPM1300-QEXX

Commit message: test: change C2 to 22uF to exercise the BOM diff
Co-Authored-By: Claude Opus 5.5 <noreply@anthropic.com>
Parts:
- C2: value 10uF -> 22uF
Changed lines of the file:
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@@
 			)
 		)
-		(property "Value" "10uF"
+		(property "Value" "22uF"
 			(at 161.29 50.8062 0)
 			(effects
