File: examples/royalblue54l-feather/sch/nRF54L15.kicad_sch (KiCad schematic)
At the start: 20 parts, among them J6 Conn_01x05_MountingPin, SW1 SW_Push, SW2 SW_Push, U1 BM15x, U4 W25Q16JVUXIQ, Y1 32.768KHz

Commit message: demo: change R5 to 4k7 to try the compare page (do not merge)
Co-Authored-By: Claude Opus 5.5 <noreply@anthropic.com>
Parts:
- R5: value 10kR -> 4k7
Changed lines of the file:
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@@
 			)
 		)
-		(property "Value" "10kR"
+		(property "Value" "4k7"
 			(at 176.53 63.4999 0)
 			(effects
