File: examples/royalblue54l-feather/RoyalBlue54L-Feather.kicad_pcb (KiCad board)
At the start: 8 copper layers, 58.4 x 22.9 mm, 71 parts, among them J1 Conn_01x16_Pin, J2 Conn_01x12_Pin, J3 USB_C_Receptacle_USB2.0_16P, J4 Conn_01x02_MountingPin, J5 Conn_01x04_MountingPin, J6 Conn_01x05_MountingPin, J8 Conn_ARM_SWD_TagConnect_TC203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, SW1 SW_Push, SW2 SW_Push, U1 BM15x, U2 nPM1300-QEXX, U3 TPD3E001DRLR, U4 W25Q16JVUXIQ, U5 nRF52833-QDXX, U6 TXB0106RGY, Y1 32.768KHz, Y2 32MHz

Commit message: test: R5 value and position (compare demo, not to merge)
Parts:
- moved R5 1.50 mm to (169.7, 113.6)
Changed lines of the file:
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@@
 (footprint "Resistor_SMD:R_0402_1005Metric"
 	(layer "F.Cu")
-	(at 169.7 112.07 180)
+	(at 169.7 113.57 180)
 	(descr "Resistor SMD 0402 (1005 Metric), square (rectangular) end terminal, IPC_7351 nominal, (Body size source: IPC-SM-782 page 72, https://www.pcb-3d.com/wordpress/wp-content/uploads/ipc-sm-782a_amendment_1_and_2.pdf), generated with kicad-footprint-generator")
 	(tags "resistor")
